File: Variante_A_LDO/Servo_Driver_A_LDO.kicad_sch (KiCad schematic)
At the start: 19 parts, among them J1 BATT 7.4V (JST-PH), J2 PWM IN 3.3V, J3 SERVO 1, J4 SERVO 2, J5 SERVO 3, U1 LM7805, U2 LM324

Commit message: PCB a foro passante per entrambe le varianti
- Variante B: LM2596T-5.0 (TO-220-5) al posto della versione SMD
- Fori di fissaggio M3 nello schema
- PCB 80x60 mm a 2 strati: piste di potenza da 1.5 mm, piano di massa
  su entrambe le facce, segnali sbrogliati con Freerouting; DRC pulito
- UUID deterministici, così schema e PCB restano collegati
- README aggiornato

Co-Authored-By: Claude Opus 5.5 <noreply@anthropic.com>
Claude-Session: https://claude.ai/code/session_01B5RPuFFwz1raQxdy9coUUD
Parts:
- added H1, H2, H3, H4: M3, MountingHole:MountingHole_3.2mm_M3, symbol Mechanical:MountingHole
Other:
- note added: "Fori di fissaggio M3"
